Commit message: add: comment to fix

File: urdf/tsukutsuku.urdf.xacro (robot description, xacro)
@@ -8,5 +8,5 @@
   <link name="base_link">
     <visual>
-      <origin xyz="0 0 0" rpy="${M_PI/2} 0 ${-M_PI/2}" />
+      <origin xyz="0 0 0" rpy="${M_PI/2} 0 ${-M_PI/2}" /> <!-- fix here  なぜかbase_linkの向きが変えられてる -->
       <geometry>
         <mesh filename="package://tsukutsuku2_description/meshes/tsukutsuku/tsukutsuku_20210820.STL" scale="1 1 1" />
@@ -19,5 +19,5 @@
   </link>
   <joint name="right_wheel_joint" type="continuous">
-    <origin xyz="0.02225 -0.215 -0.01" rpy="${-M_PI/2} 0 0" />
+    <origin xyz="0.02225 -0.215 -0.01" rpy="${-M_PI/2} 0 0" />  <!-- fix here -->
     <parent link="base_link" />
     <child link="right_wheel_link" />
@@ -28,15 +28,34 @@
   </link>
   <joint name="left_wheel_joint" type="continuous">
-    <origin xyz="0.02225 0.215 -0.01" rpy="${M_PI/2} 0 0" />
+    <origin xyz="0.02225 0.215 -0.01" rpy="${M_PI/2} 0 0" />  <!-- fix here -->
     <parent link="base_link" />
     <child link="left_wheel_link" />
     <axis xyz="0 0 1" />
   </joint>
-  <link name="caster_link"></link>
+  <!-- <link name="caster_link"></link>
   <joint name="caster_joint" type="fixed">
     <origin xyz="0.65 0 0.0" rpy="0 0 0" />
     <parent link="base_link" />
     <child link="caster_link" />
+  </joint> -->
+  <!--  ADD caster wheels !!!!!!!!!!!!!!!!!!!!! -->
+  <!-- <link name="left_caster_wheel_link">
+    <origin xyz="0 0 0" rpy="0 0 0" />
+  </link>
+  <joint name="left_caster_wheel_joint" type="continuous">
+    <origin xyz="0.65 0.215 0.0" rpy="0 0 0" />  <============= fix here
+    <parent link="base_link" />
+    <child link="left_caster_wheel_link" />
+    <axis xyz="0 0 1" />
   </joint>
+  <link name="right_caster_wheel_link">
+    <origin xyz="0 0 0" rpy="0 0 0" />
+  </link>
+  <joint name="right_caster_wheel_joint" type="continuous">
+    <origin xyz="0.65 -0.215 0.0" rpy="0 0 0" /> <============ fix here
+    <parent link="base_link" />
+    <child link="right_caster_wheel_link" />
+    <axis xyz="0 0 1" />
+  </joint> -->
   <link name="base_footprint" />
   <joint name="base_footprint_joint" type="fixed">
@@ -49,9 +68,10 @@
   </link>
   <joint name="velodyne_joint" type="fixed">
-    <origin xyz="0.27  0.00  0.827" rpy="0 0 0" />
+    <origin xyz="0.27  0.00  0.827" rpy="0 0 0" />    <!-- fix here -->
     <parent link="base_link" />
     <child link="velodyne" />
     <axis xyz="0 0 0" />
   </joint>
+  <!-- ??? -->
   <link name="hokuyo3d">
     <origin xyz="0 0 0" rpy="0 0 0" />
@@ -63,4 +83,5 @@
     <axis xyz="0 0 0" />
   </joint>
+<!--
   <link name="laser_front_left">
     <origin xyz="0 0 0" rpy="0 0 0" />
@@ -89,4 +110,32 @@
     <child link="laser_rear" />
     <axis xyz="0 0 0" />
+  </joint> -->
+  <!-- livox -->
+  <link name="livox_front_left">
+    <origin xyz="0 0 0" rpy="0 0 0" />
+  </link>
+  <joint name="livox_front_left_joint" type="fixed">
+    <origin xyz="0.67  0.16  0.26" rpy="0.0  ${M_PI} ${M_PI + M_PI/4}" /> <!-- fix here -->
+    <parent link="base_link" />
+    <child link="livox_front_left" />
+    <axis xyz="0 0 0" />
+  </joint>
+  <link name="livox_front_right">
+    <origin xyz="0 0 0" rpy="0 0 0" />
+  </link>
+  <joint name="livox_front_right_joint" type="fixed">
+    <origin xyz="0.67  -0.16  0.26" rpy="-0.0  ${M_PI} ${M_PI - M_PI/4}" /> <!-- fix here -->
+    <parent link="base_link" />
+    <child link="livox_front_right" />
+    <axis xyz="0 0 0" />
+  </joint>
+  <link name="livox_rear">
+    <origin xyz="0 0 0" rpy="0 0 0 0 0 0" />
+  </link>
+  <joint name="livox_rear_joint" type="fixed">
+    <origin xyz="-0.12  0.00  0.20" rpy="3.14159  0.00  3.14159" /> <!-- fix here -->
+    <parent link="base_link" />
+    <child link="livox_rear" />
+    <axis xyz="0 0 0" />
   </joint>
   <link name="center_camera_link">
@@ -94,5 +143,5 @@
   </link>
   <joint name="center_camera_joint" type="fixed">
-    <origin xyz="0.315  0.00  1.15" rpy="${-M_PI/2} 0 0" />
+    <origin xyz="0.315  0.00  1.15" rpy="${-M_PI/2} 0 0" /> <!-- fix here -->
     <parent link="base_link" />
     <child link="center_camera_link" />
@@ -103,5 +152,5 @@
   </link>
   <joint name="center_camera_link2center_camera_joint" type="fixed">
-    <origin xyz="0.0  0.00  0.0" rpy="0 ${M_PI/2} 0" />
+    <origin xyz="0.0  0.00  0.0" rpy="0 ${M_PI/2} 0" />  <!-- fix here??????? -->
     <parent link="center_camera_link" />
     <child link="center_camera" />
@@ -112,5 +161,5 @@
   </link>
   <joint name="imu_joint" type="fixed">
-    <origin xyz="0.376 0 0.745" rpy="${M_PI} 0 ${M_PI}" />
+    <origin xyz="0.376 0 0.745" rpy="${M_PI} 0 ${M_PI}" /> <!-- fix here -->
     <parent link="base_link" />
     <child link="imu_link" />

Commit message: fix: livox frame

File: urdf/tsukutsuku.urdf.xacro (robot description, xacro)
@@ -111,30 +111,12 @@
     <axis xyz="0 0 0" />
   </joint> -->
-  <!-- livox -->
-  <link name="livox_front_left">
+  <!-- livox (3台が1つのframeでpublishされてる 3台の配置はbase_linkから見たものになっているので tfは0,0,0) -->
+  <link name="livox">
     <origin xyz="0 0 0" rpy="0 0 0" />
   </link>
-  <joint name="livox_front_left_joint" type="fixed">
-    <origin xyz="0.67  0.16  0.26" rpy="0.0  ${M_PI} ${M_PI + M_PI/4}" /> <!-- fix here -->
+  <joint name="livox_joint" type="fixed">
+    <origin xyz="0.00  0.00  0.00" rpy="0 0 0" />
     <parent link="base_link" />
-    <child link="livox_front_left" />
-    <axis xyz="0 0 0" />
-  </joint>
-  <link name="livox_front_right">
-    <origin xyz="0 0 0" rpy="0 0 0" />
-  </link>
-  <joint name="livox_front_right_joint" type="fixed">
-    <origin xyz="0.67  -0.16  0.26" rpy="-0.0  ${M_PI} ${M_PI - M_PI/4}" /> <!-- fix here -->
-    <parent link="base_link" />
-    <child link="livox_front_right" />
-    <axis xyz="0 0 0" />
-  </joint>
-  <link name="livox_rear">
-    <origin xyz="0 0 0" rpy="0 0 0 0 0 0" />
-  </link>
-  <joint name="livox_rear_joint" type="fixed">
-    <origin xyz="-0.12  0.00  0.20" rpy="3.14159  0.00  3.14159" /> <!-- fix here -->
-    <parent link="base_link" />
-    <child link="livox_rear" />
+    <child link="livox" />
     <axis xyz="0 0 0" />
   </joint>

Commit message: preliminary

File: urdf/tsukutsuku.urdf.xacro (robot description, xacro)
@@ -15,20 +15,20 @@
     </visual>
   </link>
-  <link name="right_wheel_link">
+  <link name="rear_right_wheel_link">
       <origin xyz="0 0 0" rpy="0 0 0" />
   </link>
-  <joint name="right_wheel_joint" type="continuous">
-    <origin xyz="0.02225 -0.215 -0.01" rpy="${-M_PI/2} 0 0" />  <!-- fix here -->
+  <joint name="rear_right_wheel_joint" type="continuous">
+    <origin xyz="0 -0.2985 0" rpy="${M_PI/2} 0 0" />  <!-- fix here -->
     <parent link="base_link" />
-    <child link="right_wheel_link" />
+    <child link="rear_right_wheel_link" />
     <axis xyz="0 0 1" />
   </joint>
-  <link name="left_wheel_link">
+  <link name="rear_left_wheel_link">
         <origin xyz="0 0 0" rpy="0 0 0" />
   </link>
-  <joint name="left_wheel_joint" type="continuous">
-    <origin xyz="0.02225 0.215 -0.01" rpy="${M_PI/2} 0 0" />  <!-- fix here -->
+  <joint name="rear_left_wheel_joint" type="continuous">
+    <origin xyz="0 0.2985 0" rpy="${M_PI/2} 0 0" />  <!-- fix here -->
     <parent link="base_link" />
-    <child link="left_wheel_link" />
+    <child link="rear_left_wheel_link" />
     <axis xyz="0 0 1" />
   </joint>
@@ -40,22 +40,22 @@
   </joint> -->
   <!--  ADD caster wheels !!!!!!!!!!!!!!!!!!!!! -->
-  <!-- <link name="left_caster_wheel_link">
+  <link name="front_left_wheel_link">
     <origin xyz="0 0 0" rpy="0 0 0" />
   </link>
-  <joint name="left_caster_wheel_joint" type="continuous">
-    <origin xyz="0.65 0.215 0.0" rpy="0 0 0" />  <============= fix here
+  <joint name="front_left_wheel_joint" type="continuous">
+    <origin xyz="0.514 0.32 0.0225" rpy="${M_PI/2} 0 0" />
     <parent link="base_link" />
-    <child link="left_caster_wheel_link" />
+    <child link="front_left_wheel_link" />
     <axis xyz="0 0 1" />
   </joint>
-  <link name="right_caster_wheel_link">
+  <link name="front_right_wheel_link">
     <origin xyz="0 0 0" rpy="0 0 0" />
   </link>
-  <joint name="right_caster_wheel_joint" type="continuous">
-    <origin xyz="0.65 -0.215 0.0" rpy="0 0 0" /> <============ fix here
+  <joint name="front_right_wheel_joint" type="continuous">
+    <origin xyz="0.514 -0.32 0.0225" rpy="${M_PI/2} 0 0" />
     <parent link="base_link" />
-    <child link="right_caster_wheel_link" />
+    <child link="front_right_wheel_link" />
     <axis xyz="0 0 1" />
-  </joint> -->
+  </joint>
   <link name="base_footprint" />
   <joint name="base_footprint_joint" type="fixed">
@@ -68,55 +68,36 @@
   </link>
   <joint name="velodyne_joint" type="fixed">
-    <origin xyz="0.27  0.00  0.827" rpy="0 0 0" />    <!-- fix here -->
+    <origin xyz="0.2813  0.00  0.9265" rpy="0 0 0" />    <!-- fix here -->
     <parent link="base_link" />
     <child link="velodyne" />
     <axis xyz="0 0 0" />
   </joint>
-  <!-- ??? -->
-  <link name="hokuyo3d">
+  <!-- livox (3台が1つのframeでpublishされてる 3台の配置はbase_linkから見たものになっているので tfは0,0,0) -->
+  <link name="left_livox_link">
     <origin xyz="0 0 0" rpy="0 0 0" />
   </link>
-  <joint name="hokuyo3d_joint" type="fixed">
-    <origin xyz="0.465  0.00  0.85" rpy="0.00  0.02  -3.16" />
+  <joint name="left_livox_joint" type="fixed">
+    <origin xyz="0.7151  0.3021  0.1425" rpy="${M_PI} 0 ${-M_PI/4}" />
     <parent link="base_link" />
-    <child link="hokuyo3d" />
+    <child link="left_livox_link" />
     <axis xyz="0 0 0" />
   </joint>
-<!--
-  <link name="laser_front_left">
+  <link name="right_livox_link">
     <origin xyz="0 0 0" rpy="0 0 0" />
   </link>
-  <joint name="laser_front_left_joint" type="fixed">
-    <origin xyz="0.67  0.16  0.26" rpy="0.0  ${M_PI} ${M_PI + M_PI/4}" />
+  <joint name="right_livox_joint" type="fixed">
+    <origin xyz="0.7151  -0.3021  0.1425" rpy="${M_PI} 0 ${M_PI/4}" />
     <parent link="base_link" />
-    <child link="laser_front_left" />
+    <child link="right_livox_link" />
     <axis xyz="0 0 0" />
   </joint>
-  <link name="laser_front_right">
+  <!-- rearは後々yaw角回転の可能性あり -->
+  <link name="rear_livox_link">
     <origin xyz="0 0 0" rpy="0 0 0" />
   </link>
-  <joint name="laser_front_right_joint" type="fixed">
-    <origin xyz="0.67  -0.16  0.26" rpy="-0.0  ${M_PI} ${M_PI - M_PI/4}" />
+  <joint name="rear_livox_joint" type="fixed">
+    <origin xyz="-0.1425  0.00  0.1025" rpy="${M_PI} 0 0" />
     <parent link="base_link" />
-    <child link="laser_front_right" />
-    <axis xyz="0 0 0" />
-  </joint>
-  <link name="laser_rear">
-    <origin xyz="0 0 0" rpy="0 0 0 0 0 0" />
-  </link>
-  <joint name="laser_rear_joint" type="fixed">
-    <origin xyz="-0.12  0.00  0.20" rpy="3.14159  0.00  3.14159" />
-    <parent link="base_link" />
-    <child link="laser_rear" />
-    <axis xyz="0 0 0" />
-  </joint> -->
-  <!-- livox (3台が1つのframeでpublishされてる 3台の配置はbase_linkから見たものになっているので tfは0,0,0) -->
-  <link name="livox">
-    <origin xyz="0 0 0" rpy="0 0 0" />
-  </link>
-  <joint name="livox_joint" type="fixed">
-    <origin xyz="0.00  0.00  0.00" rpy="0 0 0" />
-    <parent link="base_link" />
-    <child link="livox" />
+    <child link="rear_livox_link" />
     <axis xyz="0 0 0" />
   </joint>
@@ -125,16 +106,7 @@
   </link>
   <joint name="center_camera_joint" type="fixed">
-    <origin xyz="0.315  0.00  1.15" rpy="${-M_PI/2} 0 0" /> <!-- fix here -->
+    <origin xyz="0.1981  0.00  1.145" rpy="0 0 0" /> <!-- fix here -->
     <parent link="base_link" />
     <child link="center_camera_link" />
-    <axis xyz="0 0 0" />
-  </joint>
-  <link name="center_camera">
-    <origin xyz="0 0 0" rpy="0 0 0" />
-  </link>
-  <joint name="center_camera_link2center_camera_joint" type="fixed">
-    <origin xyz="0.0  0.00  0.0" rpy="0 ${M_PI/2} 0" />  <!-- fix here??????? -->
-    <parent link="center_camera_link" />
-    <child link="center_camera" />
     <axis xyz="0 0 0" />
   </joint>
@@ -143,5 +115,5 @@
   </link>
   <joint name="imu_joint" type="fixed">
-    <origin xyz="0.376 0 0.745" rpy="${M_PI} 0 ${M_PI}" /> <!-- fix here -->
+    <origin xyz="0.5678 0 0.2374" rpy="${M_PI} 0 ${M_PI}" /> <!-- fix here -->
     <parent link="base_link" />
     <child link="imu_link" />

Commit message: add: livox_link(複数 frameにできない)

File: urdf/tsukutsuku.urdf.xacro (robot description, xacro)
@@ -74,4 +74,13 @@
   </joint>
   <!-- livox (3台が1つのframeでpublishされてる 3台の配置はbase_linkから見たものになっているので tfは0,0,0) -->
+  <link name="livox_link">
+    <origin xyz="0 0 0" rpy="0 0 0" />
+  </link>
+  <joint name="livox_joint" type="fixed">
+    <origin xyz="0.0  0.0  0.0" rpy="0 0 0" />
+    <parent link="base_link" />
+    <child link="livox_link" />
+    <axis xyz="0 0 0" />
+  </joint>
   <link name="left_livox_link">
     <origin xyz="0 0 0" rpy="0 0 0" />
